File: Software/SchemtaicHelper/Generated Schematic/Dell KB216t schematic.kicad_sch (KiCad schematic)
At the start: 36 parts, among them J1 Conn_01x01, J10 Conn_01x01, J100 Conn_01x01, J11 Conn_01x01, J12 Conn_01x01, J13 Conn_01x01, J14 Conn_01x01, J15 Conn_01x01, J16 Conn_01x01, J17 Conn_01x01, J18 Conn_01x01, J19 Conn_01x01, J2 Conn_01x01, J20 Conn_01x01, J21 Conn_01x01, J22 Conn_01x01, J23 Conn_01x01, J24 Conn_01x01, J25 Conn_01x01, J26 Conn_01x01, J27 Conn_01x01, J28 Conn_01x01, J3 Conn_01x01, J4 Conn_01x01, J5 Conn_01x01, J6 Conn_01x01, J7 Conn_01x01, J8 Conn_01x01, J9 Conn_01x01, M1 Conn_02x05_Odd_Even, M100 Conn_02x05_Odd_Even, M2 Conn_02x05_Odd_Even, M3 Conn_02x05_Odd_Even, M4 Conn_02x05_Odd_Even

Commit message: Dell KB212-B schematic generated
Parts:
- removed D1 (x2): Conn_02x30_Odd_Even, Connector_PinHeader_2.54mm:PinHeader_2x30_P2.54mm_Vertical, symbol Connector_Generic:Conn_02x30_Odd_Even
- removed J100: Conn_01x01, MatchBoxLibrary:Ma, symbol Connector_Generic:Conn_01x01
- removed M100: Conn_02x05_Odd_Even, Connector_PinHeader_2.54mm:PinHeader_2x05_P2.54mm_Vertical, symbol Connector_Generic:Conn_02x05_Odd_Even
- added D1: Conn_02x30_Odd_Even, Connector_PinHeader_2.54mm:PinHeader_2x30_P2.54mm_Vertical, symbol Connector_Generic:Conn_02x30_Odd_Even
Connections:
- net Pin1: now also D1.1 (Pin_1), D1.2 (Pin_2)
- net Pin10: now also D1.19 (Pin_19), D1.20 (Pin_20)
- net Pin11: now also D1.21 (Pin_21), D1.22 (Pin_22)
- net Pin12: now also D1.23 (Pin_23), D1.24 (Pin_24)
- net Pin13: now also D1.25 (Pin_25), D1.26 (Pin_26)
- net Pin14: now also D1.27 (Pin_27), D1.28 (Pin_28)
- net Pin15: now also D1.29 (Pin_29), D1.30 (Pin_30)
- net Pin16: now also D1.31 (Pin_31), D1.32 (Pin_32)
- net Pin17: now also D1.33 (Pin_33), D1.34 (Pin_34)
- net Pin18: now also D1.35 (Pin_35), D1.36 (Pin_36)
- net Pin19: now also D1.37 (Pin_37), D1.38 (Pin_38)
- net Pin2: now also D1.3 (Pin_3), D1.4 (Pin_4)
- net Pin20: now also D1.39 (Pin_39), D1.40 (Pin_40)
- net Pin21: now also D1.41 (Pin_41), D1.42 (Pin_42)
- net Pin22: now also D1.43 (Pin_43), D1.44 (Pin_44)
- net Pin23: now also D1.45 (Pin_45), D1.46 (Pin_46)
- net Pin24: now also D1.47 (Pin_47), D1.48 (Pin_48)
- net Pin25: now also D1.49 (Pin_49), D1.50 (Pin_50)
- net Pin26: now also D1.51 (Pin_51), D1.52 (Pin_52)
- net Pin27: now also D1.53 (Pin_53), D1.54 (Pin_54)
- net Pin28: now also D1.55 (Pin_55), D1.56 (Pin_56)
- net Pin29: now also D1.57 (Pin_57), D1.58 (Pin_58)
- net Pin3: now also D1.5 (Pin_5), D1.6 (Pin_6)
- net Pin30: now also D1.59 (Pin_59), D1.60 (Pin_60)
- net Pin4: now also D1.7 (Pin_7), D1.8 (Pin_8)
- net Pin5: now also D1.10 (Pin_10), D1.9 (Pin_9)
- net Pin6: now also D1.11 (Pin_11), D1.12 (Pin_12)
- net Pin7: now also D1.13 (Pin_13), D1.14 (Pin_14)
- net Pin8: now also D1.15 (Pin_15), D1.16 (Pin_16)
- net Pin9: now also D1.17 (Pin_17), D1.18 (Pin_18)
